Commit message: suru_v1_0 - v1.3

File: ROS/src/suru_v1_0/urdf/DCMachine_ChassisAssy3.urdf (robot description, URDF)
Before this commit: robot DCMachine_ChassisAssy3, 9 links, 8 joints
Joints:
- joint LDwheel_joint: type continuous -> fixed
- joint RDwheel_joint: type continuous -> fixed

Commit message: lidar laser angle filtered

File: ROS/src/suru_v1_0/urdf/DCMachine_ChassisAssy3.urdf (robot description, URDF)
Before this commit: robot DCMachine_ChassisAssy3, 9 links, 8 joints
Joints:
- joint Lidar_joint: origin xyz=0.57569 0.032864 0.20635 rpy=0 -0.087266 0 -> xyz=0.57569 0.032864 0.20635 rpy=0 0.087266 0

Commit message: backup

File: ROS/src/suru_v1_0/urdf/DCMachine_ChassisAssy3.urdf (robot description, URDF)
Before this commit: robot DCMachine_ChassisAssy3, 9 links, 8 joints
Joints:
- joint base_joint: origin xyz=0.0 0.0 0.075 rpy=0 0 3.14159 -> xyz=0.0 0.0 0.075 rpy=0 0 0
